File: Boards/uV Board/RevA/StrainGuage.sch (KiCad schematic (older format))
At the start: 0 parts

Commit message: Added a lot to the microVolt board.
Other:
- note added: "Hemobllo Strain Guage"
Changed lines of the file:
@@
 $Descr A4 11693 8268
 encoding utf-8
-Sheet 1 4
+Sheet 3 6
 Title ""
 Date ""
@@
 Comment4 ""
 $EndDescr
+Text Notes 2450 1150 0    50   ~ 0
+Hemobllo Strain Guage
+Text HLabel 2900 1350 2    50   Input ~ 0
+5V
+Text HLabel 2900 1550 2    50   Input ~ 0
+GND
+Text HLabel 2900 1450 2    50   Input ~ 0
+Strain_Out
+Text Label 2350 1350 2    50   ~ 0
+Strain_In_Hi
+Text Label 2350 1550 2    50   ~ 0
+Strain_In_Lo
 $EndSCHEMATC
