File: Boards/ADC Board/RevA/Button Inputs.sch (KiCad schematic (older format))
At the start: 0 parts

Commit message: Copied controller board from micro board to ADC board. Created pull up/down sheets and populated them.
Also copied over main set of header pins into ADC sheet.
Parts:
- added J?: Conn_02x10_Counter_Clockwise, symbol Connector_Generic:Conn_02x10_Counter_Clockwise
Changed lines of the file:
@@
 $Descr A4 11693 8268
 encoding utf-8
-Sheet 4 4
+Sheet 4 7
 Title ""
 Date ""
@@
 Comment4 ""
 $EndDescr
+$Comp
+L Connector_Generic:Conn_02x10_Counter_Clockwise J?
+U 1 1 61602C7D
+P 2250 1400
+F 0 "J?" H 2300 2017 50  0000 C CNN
+F 1 "Conn_02x10_Counter_Clockwise" H 2300 1926 50  0000 C CNN
+F 2 "" H 2250 1400 50  0001 C CNN
+F 3 "~" H 2250 1400 50  0001 C CNN
+	1    2250 1400
+	1    0    0    -1
+$EndComp
+Text HLabel 5600 550  2    50   Input ~ 0
+5V
+Text HLabel 5600 650  2    50   Input ~ 0
+GND
+Text HLabel 5600 750  2    50   Input ~ 0
+3.3V
+Text Label 5600 550  2    50   ~ 0
+5V
+Text Label 5600 650  2    50   ~ 0
+GND
+Text Label 5600 750  2    50   ~ 0
+3.3V
 $EndSCHEMATC
