File: Boards/ADC Board/RevA1/controller.sch (KiCad schematic (older format))
At the start: 3 parts, among them J11 Arduino Nano, J12 Arduino Nano, J13 Extra Pins

Commit message: Moved around components on the ADC board PCB. Assigned footprints to microVolt board components.
Tried to add 6-pin spring connector to custom schematics list.
Parts:
- J11: value Arduino Nano -> Arduino Nano L
- J12: value Arduino Nano -> Arduino Nano R
Changed lines of the file:
@@
 P 1600 1550
 F 0 "J11" H 2050 1500 50  0000 L CNN
-F 1 "Arduino Nano" H 1850 1400 50  0000 L CNN
+F 1 "Arduino Nano L" H 1850 1400 50  0000 L CNN
 F 2 "Connector_PinSocket_2.54mm:PinSocket_1x15_P2.54mm_Vertical" H 1600 1550 50  0001 C CNN
 F 3 "~" H 1600 1550 50  0001 C CNN
@@
 P 2800 1550
 F 0 "J12" H 3150 2000 50  0000 L CNN
-F 1 "Arduino Nano" H 2950 1900 50  0000 L CNN
+F 1 "Arduino Nano R" H 2950 1900 50  0000 L CNN
 F 2 "Connector_PinSocket_2.54mm:PinSocket_1x15_P2.54mm_Vertical" H 2800 1550 50  0001 C CNN
 F 3 "~" H 2800 1550 50  0001 C CNN
