File: Boards/Breadboard_Testbed/RevA/Breadboard-Testbed.sch (KiCad schematic (older format))
At the start: 11 parts, among them J1 main_conn_10, J2 main_conn_12

Commit message: Finished Breadboard-Testbed RevA Schematic
Parts:
- removed D1: LED, LED_SMD:LED_1812_4532Metric, symbol Device:LED
- removed R5: 350?, Resistor_SMD:R_0603_1608Metric, symbol Device:R_US
- added J? (x2): Arduino-left, symbol Connector_Generic:Conn_02x15_Counter_Clockwise
- added J? (x2): Arduino-right, symbol Connector_Generic:Conn_02x15_Counter_Clockwise
Connections:
- net 3v3: no longer J1.17 (Pin_17), J?.17 (Pin_17), J?.4 (Pin_4)
- net 5v: no longer J1.4 (Pin_4), J?.17 (Pin_17), J?.4 (Pin_4)
- net NC: now also J?.21 (Pin_21), J?.4 (Pin_4); no longer J?.21 (Pin_21), J?.4 (Pin_4)
- net gnd: no longer J1.14 (Pin_14), J1.20 (Pin_20), J1.9 (Pin_9), J2.10 (Pin_10), J2.14 (Pin_14), J2.19 (Pin_19), J2.5 (Pin_5), J?.1 (Pin_1), J?.10 (Pin_10), J?.11 (Pin_11), J?.12 (Pin_12), J?.14 (Pin_14), J?.14 (Pin_14), J?.15 (Pin_15), J?.19 (Pin_19), J?.20 (Pin_20), J?.20 (Pin_20), J?.5 (Pin_5), J?.6 (Pin_6), J?.7 (Pin_7), J?.9 (Pin_9)
- net gpio10: now also J?.17 (Pin_17), J?.8 (Pin_8); no longer J?.17 (Pin_17), J?.8 (Pin_8)
- net gpio2: now also J?.16 (Pin_16), J?.9 (Pin_9); no longer J?.16 (Pin_16), J?.9 (Pin_9)
- net gpio3: now also J?.11 (Pin_11), J?.14 (Pin_14); no longer J?.11 (Pin_11), J?.14 (Pin_14)
- net gpio4: now also J?.12 (Pin_12), J?.13 (Pin_13); no longer J?.12 (Pin_12), J?.13 (Pin_13)
- net gpio5: now also J?.12 (Pin_12), J?.13 (Pin_13); no longer J?.12 (Pin_12), J?.13 (Pin_13)
- net gpio9: now also J?.2 (Pin_2), J?.23 (Pin_23); no longer J?.2 (Pin_2), J?.23 (Pin_23)
- net miso: now also J?.1 (Pin_1), J?.24 (Pin_24); no longer J?.1 (Pin_1), J?.24 (Pin_24)
- net miso2: now also J?.18 (Pin_18), J?.7 (Pin_7); no longer J?.18 (Pin_18), J?.7 (Pin_7)
- net miso2_pwm: now also J?.10 (Pin_10), J?.15 (Pin_15); no longer J?.10 (Pin_10), J?.15 (Pin_15)
- net reset: now also J?.22 (Pin_22), J?.3 (Pin_3); no longer J?.22 (Pin_22), J?.3 (Pin_3)
- net scl: now also J?.17 (Pin_17), J?.8 (Pin_8); no longer J?.17 (Pin_17), J?.8 (Pin_8)
- net sclk: now also J?.22 (Pin_22), J?.3 (Pin_3); no longer J?.22 (Pin_22), J?.3 (Pin_3)
- net sclk2: now also J?.20 (Pin_20), J?.5 (Pin_5); no longer J?.20 (Pin_20), J?.5 (Pin_5)
- net sda: now also J?.18 (Pin_18), J?.7 (Pin_7); no longer J?.18 (Pin_18), J?.7 (Pin_7)
- net spi2_ce2: now also J?.16 (Pin_16), J?.9 (Pin_9); no longer J?.16 (Pin_16), J?.9 (Pin_9)
- net spi_ce0: now also J?.21 (Pin_21), J?.4 (Pin_4); no longer J?.21 (Pin_21), J?.4 (Pin_4)
- net spi_ce1: now also J?.19 (Pin_19), J?.6 (Pin_6); no longer J?.19 (Pin_19), J?.6 (Pin_6)
- net vcc: now also J?.2 (Pin_2), J?.23 (Pin_23); no longer J2.24 (Pin_24), J?.1 (Pin_1), J?.2 (Pin_2), J?.23 (Pin_23), J?.24 (Pin_24)
- new net: J?.1 (Pin_1), J?.30 (Pin_30) (x4)
- new net: J?.10 (Pin_10), J?.21 (Pin_21) (x4)
- new net: J?.11 (Pin_11), J?.20 (Pin_20) (x4)
- new net: J?.12 (Pin_12), J?.19 (Pin_19) (x4)
- new net: J?.13 (Pin_13), J?.18 (Pin_18) (x4)
- new net: J?.14 (Pin_14), J?.17 (Pin_17) (x4)
- new net: J?.15 (Pin_15), J?.16 (Pin_16) (x4)
- new net: J?.2 (Pin_2), J?.29 (Pin_29) (x4)
- new net: J?.22 (Pin_22), J?.9 (Pin_9) (x4)
- new net: J?.23 (Pin_23), J?.8 (Pin_8) (x4)
- new net: J?.24 (Pin_24), J?.7 (Pin_7) (x4)
- new net: J?.25 (Pin_25), J?.6 (Pin_6) (x4)
- new net: J?.26 (Pin_26), J?.5 (Pin_5) (x4)
- new net: J?.27 (Pin_27), J?.4 (Pin_4) (x4)
- new net: J?.28 (Pin_28), J?.3 (Pin_3) (x4)
- new net 3v3_2: J1.17 (Pin_17), J?.17 (Pin_17), J?.4 (Pin_4)
- new net 5v2: J1.4 (Pin_4), J?.17 (Pin_17), J?.4 (Pin_4)
- new net gnd2: J1.9 (Pin_9), J?.12 (Pin_12), J?.9 (Pin_9)
- new net gnd3: J1.14 (Pin_14), J?.14 (Pin_14), J?.7 (Pin_7)
- new net gnd4: J1.20 (Pin_20), J?.1 (Pin_1), J?.20 (Pin_20)
- new net gnd_: J2.19 (Pin_19), J?.19 (Pin_19), J?.6 (Pin_6)
- new net gnd_1: J2.14 (Pin_14), J?.11 (Pin_11), J?.14 (Pin_14)
- new net gnd_2: J2.10 (Pin_10), J?.10 (Pin_10), J?.15 (Pin_15)
- new net gnd_3: J2.5 (Pin_5), J?.20 (Pin_20), J?.5 (Pin_5)
- new net vcc1: J2.24 (Pin_24), J?.1 (Pin_1), J?.24 (Pin_24)
Other:
- moved on the sheet: H?

Commit message: Generated Netlist for Breadboard-Testbed
Parts:
- H1: renamed from H?; footprint (none) -> MountingHole:MountingHole_2.5mm
- J10, J11, J6, J7: renamed from J?; footprint (none) -> Connector_PinHeader_2.54mm:PinHeader_2x15_P2.54mm_Vertical
- gave numbers to parts that had none: 6
Changed lines of the file:
@@
 +20
 $Comp
-L Connector_Generic:Conn_02x12_Counter_Clockwise J?
+L Connector_Generic:Conn_02x12_Counter_Clockwise J12
 U 1 1 61FD41D1
 P 10000 5350
-F 0 "J?" H 10050 6067 50  0000 C CNN
+F 0 "J12" H 10050 6067 50  0000 C CNN
 F 1 "Conn_02x12_Counter_Clockwise" H 10050 5976 50  0000 C CNN
 F 2 "Connector_PinHeader_2.54mm:PinHeader_2x12_P2.54mm_Vertical" H 10000 5350 50  0001 C CNN
@@
 NC
 $Comp
-L Connector_Generic:Conn_02x10_Counter_Clockwise J?
+L Connector_Generic:Conn_02x10_Counter_Clockwise J5
 U 1 1 61FF84C4
 P 5600 1700
-F 0 "J?" H 5650 2317 50  0000 C CNN
+F 0 "J5" H 5650 2317 50  0000 C CNN
 F 1 "Conn_02x10_Counter_Clockwise" H 5650 2226 50  0000 C CNN
 F 2 "Connector_PinHeader_2.54mm:PinHeader_2x10_P2.54mm_Vertical" H 5600 1700 50  0001 C CNN
@@
 $EndComp
 $Comp
-L Connector_Generic:Conn_02x10_Counter_Clockwise J?
+L Connector_Generic:Conn_02x10_Counter_Clockwise J8
 U 1 1 61FFAAA2
 P 7750 1700
-F 0 "J?" H 7800 2317 50  0000 C CNN
+F 0 "J8" H 7800 2317 50  0000 C CNN
 F 1 "Conn_02x10_Counter_Clockwise" H 7800 2226 50  0000 C CNN
 F 2 "Connector_PinHeader_2.54mm:PinHeader_2x10_P2.54mm_Vertical" H 7750 1700 50  0001 C CNN
@@
 $EndComp
 $Comp
-L Connector_Generic:Conn_02x10_Counter_Clockwise J?
+L Connector_Generic:Conn_02x10_Counter_Clockwise J3
 U 1 1 62008AB1
 P 3050 3200
-F 0 "J?" H 3100 3817 50  0000 C CNN
+F 0 "J3" H 3100 3817 50  0000 C CNN
 F 1 "Conn_02x10_Counter_Clockwise" H 3100 3726 50  0000 C CNN
 F 2 "Connector_PinHeader_2.54mm:PinHeader_2x10_P2.54mm_Vertical" H 3050 3200 50  0001 C CNN
@@
 $EndComp
 $Comp
-L Connector_Generic:Conn_02x10_Counter_Clockwise J?
+L Connector_Generic:Conn_02x10_Counter_Clockwise J4
 U 1 1 6200A2AB
 P 3850 3200
-F 0 "J?" H 3900 3817 50  0000 C CNN
+F 0 "J4" H 3900 3817 50  0000 C CNN
 F 1 "Conn_02x10_Counter_Clockwise" H 3900 3726 50  0000 C CNN
 F 2 "Connector_PinHeader_2.54mm:PinHeader_2x10_P2.54mm_Vertical" H 3850 3200 50  0001 C CNN
@@
 Connection ~ 3350 3700
 $Comp
-L Mechanical:MountingHole H?
+L Mechanical:MountingHole H1
 U 1 1 620171F6
 P 1150 4900
-F 0 "H?" H 1250 4946 50  0000 L CNN
+F 0 "H1" H 1250 4946 50  0000 L CNN
 F 1 "CMH" H 1250 4855 50  0000 L CNN
-F 2 "" H 1150 4900 50  0001 C CNN
+F 2 "MountingHole:MountingHole_2.5mm" H 1150 4900 50  0001 C CNN
 F 3 "~" H 1150 4900 50  0001 C CNN
 	1    1150 4900
@@
 $EndComp
 $Comp
-L Connector_Generic:Conn_02x15_Counter_Clockwise J?
+L Connector_Generic:Conn_02x15_Counter_Clockwise J6
 U 1 1 62019DEC
 P 6500 3400
-F 0 "J?" H 6550 4317 50  0000 C CNN
+F 0 "J6" H 6550 4317 50  0000 C CNN
 F 1 "Arduino-left" H 6550 4226 50  0000 C CNN
-F 2 "" H 6500 3400 50  0001 C CNN
+F 2 "Connector_PinHeader_2.54mm:PinHeader_2x15_P2.54mm_Vertical" H 6500 3400 50  0001 C CNN
 F 3 "~" H 6500 3400 50  0001 C CNN
 	1    6500 3400
@@
 $EndComp
 $Comp
-L Connector_Generic:Conn_02x15_Counter_Clockwise J?
+L Connector_Generic:Conn_02x15_Counter_Clockwise J7
 U 1 1 6203836E
 P 7000 3400
-F 0 "J?" H 7050 4317 50  0000 C CNN
+F 0 "J7" H 7050 4317 50  0000 C CNN
 F 1 "Arduino-left" H 7050 4226 50  0000 C CNN
-F 2 "" H 7000 3400 50  0001 C CNN
+F 2 "Connector_PinHeader_2.54mm:PinHeader_2x15_P2.54mm_Vertical" H 7000 3400 50  0001 C CNN
 F 3 "~" H 7000 3400 50  0001 C CNN
 	1    7000 3400
@@
 	6300 4100 7300 4100
 $Comp
-L Connector_Generic:Conn_02x15_Counter_Clockwise J?
+L Connector_Generic:Conn_02x15_Counter_Clockwise J10
 U 1 1 6204A5F5
 P 8100 3350
-F 0 "J?" H 8150 4267 50  0000 C CNN
+F 0 "J10" H 8150 4267 50  0000 C CNN
 F 1 "Arduino-right" H 8150 4176 50  0000 C CNN
-F 2 "" H 8100 3350 50  0001 C CNN
+F 2 "Connector_PinHeader_2.54mm:PinHeader_2x15_P2.54mm_Vertical" H 8100 3350 50  0001 C CNN
 F 3 "~" H 8100 3350 50  0001 C CNN
 	1    8100 3350
@@
 $EndComp
 $Comp
-L Connector_Generic:Conn_02x15_Counter_Clockwise J?
+L Connector_Generic:Conn_02x15_Counter_Clockwise J11
 U 1 1 6204A5FB
 P 8600 3350
-F 0 "J?" H 8650 4267 50  0000 C CNN
+F 0 "J11" H 8650 4267 50  0000 C CNN
 F 1 "Arduino-right" H 8650 4176 50  0000 C CNN
-F 2 "" H 8600 3350 50  0001 C CNN
+F 2 "Connector_PinHeader_2.54mm:PinHeader_2x15_P2.54mm_Vertical" H 8600 3350 50  0001 C CNN
 F 3 "~" H 8600 3350 50  0001 C CNN
 	1    8600 3350
@@
 gpio 10
 $Comp
-L Connector_Generic:Conn_02x12_Counter_Clockwise J?
+L Connector_Generic:Conn_02x12_Counter_Clockwise J9
 U 1 1 61FD1A5A
 P 7750 5350
-F 0 "J?" H 7800 6067 50  0000 C CNN
+F 0 "J9" H 7800 6067 50  0000 C CNN
 F 1 "Conn_02x12_Counter_Clockwise" H 7800 5976 50  0000 C CNN
 F 2 "Connector_PinHeader_2.54mm:PinHeader_2x12_P2.54mm_Vertical" H 7750 5350 50  0001 C CNN

Commit message: Fixed Breadboard-Testbed RevA arrangement, need to fix pi lineup
Parts:
- J1, J3, J4, J5, J8: symbol Connector_Generic:Conn_02x10_Counter_Clockwise -> Connector_Generic:Conn_02x10_Odd_Even
- J10, J11, J6, J7: symbol Connector_Generic:Conn_02x15_Counter_Clockwise -> Connector_Generic:Conn_02x15_Odd_Even
- J12, J2, J9: symbol Connector_Generic:Conn_02x12_Counter_Clockwise -> Connector_Generic:Conn_02x12_Odd_Even
Connections:
- net 3v3: now also J5.2 (Pin_2); no longer J5.20 (Pin_20)
- net 3v3_2: now also J1.8 (Pin_8), J8.7 (Pin_7), J8.8 (Pin_8); no longer J1.17 (Pin_17), J8.17 (Pin_17), J8.4 (Pin_4)
- net 5v: now also J1.3 (Pin_3), J5.3 (Pin_3), J5.4 (Pin_4); no longer J1.2 (Pin_2), J5.19 (Pin_19), J5.2 (Pin_2)
- net 5v2: now also J1.7 (Pin_7), J5.7 (Pin_7), J5.8 (Pin_8); no longer J1.4 (Pin_4), J5.17 (Pin_17), J5.4 (Pin_4)
- net NC: now also J2.8 (Pin_8), J9.7 (Pin_7), J9.8 (Pin_8); no longer J2.21 (Pin_21), J9.21 (Pin_21), J9.4 (Pin_4)
- net gnd: now also J1.11 (Pin_11), J5.11 (Pin_11), J5.12 (Pin_12); no longer J1.6 (Pin_6), J5.15 (Pin_15), J5.6 (Pin_6)
- net gnd2: now also J1.17 (Pin_17), J5.17 (Pin_17), J5.18 (Pin_18); no longer J1.9 (Pin_9), J5.12 (Pin_12), J5.9 (Pin_9)
- net gnd3: now also J8.13 (Pin_13); no longer J8.7 (Pin_7)
- net gnd4: now also J1.2 (Pin_2), J8.2 (Pin_2); no longer J1.20 (Pin_20), J8.20 (Pin_20)
- net gnd_: now also J2.12 (Pin_12), J9.11 (Pin_11), J9.12 (Pin_12); no longer J2.19 (Pin_19), J9.19 (Pin_19), J9.6 (Pin_6)
- net gnd_1: now also J2.22 (Pin_22), J9.21 (Pin_21), J9.22 (Pin_22); no longer J2.14 (Pin_14), J9.11 (Pin_11), J9.14 (Pin_14)
- net gnd_2: now also J12.19 (Pin_19), J12.20 (Pin_20), J2.19 (Pin_19); no longer J12.10 (Pin_10), J12.15 (Pin_15), J2.10 (Pin_10)
- net gnd_3: now also J12.10 (Pin_10), J12.9 (Pin_9), J2.9 (Pin_9); no longer J12.20 (Pin_20), J12.5 (Pin_5), J2.5 (Pin_5)
- net gpio1: now also J1.13 (Pin_13), J5.13 (Pin_13); no longer J1.7 (Pin_7), J5.7 (Pin_7)
- net gpio10: now also J2.16 (Pin_16), J9.15 (Pin_15), J9.16 (Pin_16); no longer J2.17 (Pin_17), J9.17 (Pin_17), J9.8 (Pin_8)
- net gpio11: now also J1.16 (Pin_16), J8.15 (Pin_15), J8.16 (Pin_16); no longer J1.13 (Pin_13), J8.13 (Pin_13), J8.8 (Pin_8)
- net gpio2: now also J12.17 (Pin_17), J12.18 (Pin_18), J2.17 (Pin_17); no longer J12.16 (Pin_16), J12.9 (Pin_9), J2.9 (Pin_9)
- net gpio3: now also J12.21 (Pin_21), J12.22 (Pin_22), J2.21 (Pin_21); no longer J12.11 (Pin_11), J12.14 (Pin_14), J2.11 (Pin_11)
- net gpio4: now also J12.23 (Pin_23), J12.24 (Pin_24), J2.23 (Pin_23); no longer J12.12 (Pin_12), J12.13 (Pin_13), J2.12 (Pin_12)
- net gpio5: now also J2.24 (Pin_24), J9.23 (Pin_23), J9.24 (Pin_24); no longer J2.13 (Pin_13), J9.12 (Pin_12), J9.13 (Pin_13)
- net gpio6: now also J1.12 (Pin_12), J8.11 (Pin_11), J8.12 (Pin_12); no longer J1.15 (Pin_15), J8.15 (Pin_15), J8.6 (Pin_6)
- net gpio7: now also J1.10 (Pin_10), J8.10 (Pin_10), J8.9 (Pin_9); no longer J1.16 (Pin_16), J8.16 (Pin_16), J8.5 (Pin_5)
- net gpio8: now also J1.6 (Pin_6), J8.5 (Pin_5), J8.6 (Pin_6); no longer J1.18 (Pin_18), J8.18 (Pin_18), J8.3 (Pin_3)
- net gpio9: now also J12.3 (Pin_3), J12.4 (Pin_4), J2.3 (Pin_3); no longer J12.2 (Pin_2), J12.23 (Pin_23), J2.2 (Pin_2)
- net miso: now also J12.2 (Pin_2); no longer J12.24 (Pin_24)
- net miso2: now also J2.14 (Pin_14), J9.13 (Pin_13), J9.14 (Pin_14); no longer J2.18 (Pin_18), J9.18 (Pin_18), J9.7 (Pin_7)
- net miso2_pwm: now also J2.20 (Pin_20), J9.19 (Pin_19), J9.20 (Pin_20); no longer J2.15 (Pin_15), J9.10 (Pin_10), J9.15 (Pin_15)
- net mosi: now also J1.4 (Pin_4), J8.3 (Pin_3), J8.4 (Pin_4); no longer J1.19 (Pin_19), J8.19 (Pin_19), J8.2 (Pin_2)
- net reset: now also J2.6 (Pin_6), J9.5 (Pin_5), J9.6 (Pin_6); no longer J2.22 (Pin_22), J9.22 (Pin_22), J9.3 (Pin_3)
- net scl: now also J12.15 (Pin_15), J12.16 (Pin_16), J2.15 (Pin_15); no longer J12.17 (Pin_17), J12.8 (Pin_8), J2.8 (Pin_8)
- net scl2: now also J1.9 (Pin_9), J5.10 (Pin_10), J5.9 (Pin_9); no longer J1.5 (Pin_5), J5.16 (Pin_16), J5.5 (Pin_5)
- net sclk: now also J12.5 (Pin_5), J12.6 (Pin_6), J2.5 (Pin_5); no longer J12.22 (Pin_22), J12.3 (Pin_3), J2.3 (Pin_3)
- net sclk2: now also J2.10 (Pin_10), J9.10 (Pin_10), J9.9 (Pin_9); no longer J2.20 (Pin_20), J9.20 (Pin_20), J9.5 (Pin_5)
- net sda: now also J12.13 (Pin_13), J12.14 (Pin_14), J2.13 (Pin_13); no longer J12.18 (Pin_18), J12.7 (Pin_7), J2.7 (Pin_7)
- net sda2: now also J1.5 (Pin_5), J5.5 (Pin_5), J5.6 (Pin_6); no longer J1.3 (Pin_3), J5.18 (Pin_18), J5.3 (Pin_3)
- net spi2_ce0: now also J1.18 (Pin_18), J8.17 (Pin_17), J8.18 (Pin_18); no longer J1.12 (Pin_12), J8.12 (Pin_12), J8.9 (Pin_9)
- net spi2_ce1: now also J1.20 (Pin_20), J8.19 (Pin_19), J8.20 (Pin_20); no longer J1.11 (Pin_11), J8.10 (Pin_10), J8.11 (Pin_11)
- net spi2_ce2: now also J2.18 (Pin_18), J9.17 (Pin_17), J9.18 (Pin_18); no longer J2.16 (Pin_16), J9.16 (Pin_16), J9.9 (Pin_9)
- net spi_ce0: now also J12.7 (Pin_7), J12.8 (Pin_8), J2.7 (Pin_7); no longer J12.21 (Pin_21), J12.4 (Pin_4), J2.4 (Pin_4)
- net spi_ce1: now also J12.11 (Pin_11), J12.12 (Pin_12), J2.11 (Pin_11); no longer J12.19 (Pin_19), J12.6 (Pin_6), J2.6 (Pin_6)
- net uart_rx: now also J1.19 (Pin_19), J5.19 (Pin_19), J5.20 (Pin_20); no longer J1.10 (Pin_10), J5.10 (Pin_10), J5.11 (Pin_11)
- net uart_tx: now also J1.15 (Pin_15), J5.15 (Pin_15), J5.16 (Pin_16); no longer J1.8 (Pin_8), J5.13 (Pin_13), J5.8 (Pin_8)
- net vcc: now also J2.4 (Pin_4), J9.3 (Pin_3), J9.4 (Pin_4); no longer J2.23 (Pin_23), J9.2 (Pin_2), J9.23 (Pin_23)
- net vcc1: now also J2.2 (Pin_2), J9.2 (Pin_2); no longer J2.24 (Pin_24), J9.24 (Pin_24)
- net at J3.1 (Pin_1), J4.1 (Pin_1): now also J3.2 (Pin_2), J4.2 (Pin_2); no longer J3.20 (Pin_20), J4.20 (Pin_20)
- net at J3.10 (Pin_10), J4.10 (Pin_10): now also J3.9 (Pin_9), J4.9 (Pin_9); no longer J3.11 (Pin_11), J4.11 (Pin_11)
- net at J3.12 (Pin_12), J4.12 (Pin_12): now also J3.11 (Pin_11), J4.11 (Pin_11); no longer J3.9 (Pin_9), J4.9 (Pin_9)
- net at J3.13 (Pin_13), J4.13 (Pin_13): now also J3.14 (Pin_14), J4.14 (Pin_14); no longer J3.8 (Pin_8), J4.8 (Pin_8)
- net at J3.7 (Pin_7), J4.7 (Pin_7): now also J3.8 (Pin_8), J4.8 (Pin_8); no longer J3.14 (Pin_14), J4.14 (Pin_14)
- net at J3.15 (Pin_15), J4.15 (Pin_15): now also J3.16 (Pin_16), J4.16 (Pin_16); no longer J3.6 (Pin_6), J4.6 (Pin_6)
- net at J3.5 (Pin_5), J4.5 (Pin_5): now also J3.6 (Pin_6), J4.6 (Pin_6); no longer J3.16 (Pin_16), J4.16 (Pin_16)
- net at J3.17 (Pin_17), J4.17 (Pin_17): now also J3.18 (Pin_18), J4.18 (Pin_18); no longer J3.4 (Pin_4), J4.4 (Pin_4)
- net at J3.3 (Pin_3), J4.3 (Pin_3): now also J3.4 (Pin_4), J4.4 (Pin_4); no longer J3.18 (Pin_18), J4.18 (Pin_18)
- net at J3.19 (Pin_19), J4.19 (Pin_19): now also J3.20 (Pin_20), J4.20 (Pin_20); no longer J3.2 (Pin_2), J4.2 (Pin_2)
- net at J6.1 (Pin_1): now also J7.2 (Pin_2); no longer J7.30 (Pin_30)
- net at J6.10 (Pin_10): now also J7.9 (Pin_9); no longer J7.21 (Pin_21)
- net at J6.11 (Pin_11): now also J7.12 (Pin_12); no longer J7.20 (Pin_20)
- net at J6.12 (Pin_12): now also J7.11 (Pin_11); no longer J7.19 (Pin_19)
- net at J6.13 (Pin_13): now also J7.14 (Pin_14); no longer J7.18 (Pin_18)
- net at J6.14 (Pin_14): now also J7.13 (Pin_13); no longer J7.17 (Pin_17)
- net at J6.17 (Pin_17): now also J7.18 (Pin_18); no longer J7.14 (Pin_14)
- net at J6.18 (Pin_18): now also J7.17 (Pin_17); no longer J7.13 (Pin_13)
- net at J6.19 (Pin_19): now also J7.20 (Pin_20); no longer J7.12 (Pin_12)
- net at J6.2 (Pin_2): now also J7.1 (Pin_1); no longer J7.29 (Pin_29)
- net at J6.20 (Pin_20): now also J7.19 (Pin_19); no longer J7.11 (Pin_11)
- net at J6.21 (Pin_21): now also J7.22 (Pin_22); no longer J7.10 (Pin_10)
- net at J6.22 (Pin_22): now also J7.21 (Pin_21); no longer J7.9 (Pin_9)
- net at J6.23 (Pin_23): now also J7.24 (Pin_24); no longer J7.8 (Pin_8)
- net at J6.24 (Pin_24): now also J7.23 (Pin_23); no longer J7.7 (Pin_7)
- net at J6.25 (Pin_25): now also J7.26 (Pin_26); no longer J7.6 (Pin_6)
- net at J6.26 (Pin_26): now also J7.25 (Pin_25); no longer J7.5 (Pin_5)
- net at J6.27 (Pin_27): now also J7.28 (Pin_28); no longer J7.4 (Pin_4)
- net at J6.28 (Pin_28): now also J7.27 (Pin_27); no longer J7.3 (Pin_3)
- net at J6.29 (Pin_29): now also J7.30 (Pin_30); no longer J7.2 (Pin_2)
- net at J6.3 (Pin_3): now also J7.4 (Pin_4); no longer J7.28 (Pin_28)
- net at J6.30 (Pin_30): now also J7.29 (Pin_29); no longer J7.1 (Pin_1)
- net at J6.4 (Pin_4): now also J7.3 (Pin_3); no longer J7.27 (Pin_27)
- net at J6.5 (Pin_5): now also J7.6 (Pin_6); no longer J7.26 (Pin_26)
- net at J6.6 (Pin_6): now also J7.5 (Pin_5); no longer J7.25 (Pin_25)
- net at J6.7 (Pin_7): now also J7.8 (Pin_8); no longer J7.24 (Pin_24)
- net at J6.8 (Pin_8): now also J7.7 (Pin_7); no longer J7.23 (Pin_23)
- net at J6.9 (Pin_9): now also J7.10 (Pin_10); no longer J7.22 (Pin_22)
- net at J10.1 (Pin_1): now also J11.2 (Pin_2); no longer J11.30 (Pin_30)
- net at J10.10 (Pin_10): now also J11.9 (Pin_9); no longer J11.21 (Pin_21)
- net at J10.11 (Pin_11): now also J11.12 (Pin_12); no longer J11.20 (Pin_20)
- net at J10.12 (Pin_12): now also J11.11 (Pin_11); no longer J11.19 (Pin_19)
- net at J10.13 (Pin_13): now also J11.14 (Pin_14); no longer J11.18 (Pin_18)
- net at J10.14 (Pin_14): now also J11.13 (Pin_13); no longer J11.17 (Pin_17)
- net at J10.17 (Pin_17): now also J11.18 (Pin_18); no longer J11.14 (Pin_14)
- net at J10.18 (Pin_18): now also J11.17 (Pin_17); no longer J11.13 (Pin_13)
- net at J10.19 (Pin_19): now also J11.20 (Pin_20); no longer J11.12 (Pin_12)
- net at J10.2 (Pin_2): now also J11.1 (Pin_1); no longer J11.29 (Pin_29)
- net at J10.20 (Pin_20): now also J11.19 (Pin_19); no longer J11.11 (Pin_11)
- net at J10.21 (Pin_21): now also J11.22 (Pin_22); no longer J11.10 (Pin_10)
- net at J10.22 (Pin_22): now also J11.21 (Pin_21); no longer J11.9 (Pin_9)
- net at J10.23 (Pin_23): now also J11.24 (Pin_24); no longer J11.8 (Pin_8)
- net at J10.24 (Pin_24): now also J11.23 (Pin_23); no longer J11.7 (Pin_7)
- net at J10.25 (Pin_25): now also J11.26 (Pin_26); no longer J11.6 (Pin_6)
- net at J10.26 (Pin_26): now also J11.25 (Pin_25); no longer J11.5 (Pin_5)
- net at J10.27 (Pin_27): now also J11.28 (Pin_28); no longer J11.4 (Pin_4)
- net at J10.28 (Pin_28): now also J11.27 (Pin_27); no longer J11.3 (Pin_3)
- net at J10.29 (Pin_29): now also J11.30 (Pin_30); no longer J11.2 (Pin_2)
- net at J10.3 (Pin_3): now also J11.4 (Pin_4); no longer J11.28 (Pin_28)
- net at J10.30 (Pin_30): now also J11.29 (Pin_29); no longer J11.1 (Pin_1)
- net at J10.4 (Pin_4): now also J11.3 (Pin_3); no longer J11.27 (Pin_27)
- net at J10.5 (Pin_5): now also J11.6 (Pin_6); no longer J11.26 (Pin_26)
- net at J10.6 (Pin_6): now also J11.5 (Pin_5); no longer J11.25 (Pin_25)
- net at J10.7 (Pin_7): now also J11.8 (Pin_8); no longer J11.24 (Pin_24)
- net at J10.8 (Pin_8): now also J11.7 (Pin_7); no longer J11.23 (Pin_23)
- net at J10.9 (Pin_9): now also J11.10 (Pin_10); no longer J11.22 (Pin_22)
Changed lines of the file:
@@
 gpio 0
 $Comp
-L Connector_Generic:Conn_02x10_Counter_Clockwise J1
+L Connector_Generic:Conn_02x10_Odd_Even J1
 U 1 1 6160E35B
 P 1900 1750
@@
 $EndComp
 $Comp
-L Connector_Generic:Conn_02x12_Counter_Clockwise J2
+L Connector_Generic:Conn_02x12_Odd_Even J2
 U 1 1 6160FED6
 P 4300 5300
@@
 +20
 $Comp
-L Connector_Generic:Conn_02x12_Counter_Clockwise J12
+L Connector_Generic:Conn_02x12_Odd_Even J12
 U 1 1 61FD41D1
 P 10000 5350
@@
 NC
 $Comp
-L Connector_Generic:Conn_02x10_Counter_Clockwise J5
+L Connector_Generic:Conn_02x10_Odd_Even J5
 U 1 1 61FF84C4
 P 5600 1700
@@
 $EndComp
 $Comp
-L Connector_Generic:Conn_02x10_Counter_Clockwise J8
+L Connector_Generic:Conn_02x10_Odd_Even J8
 U 1 1 61FFAAA2
 P 7750 1700
@@
 $EndComp
 $Comp
-L Connector_Generic:Conn_02x10_Counter_Clockwise J3
+L Connector_Generic:Conn_02x10_Odd_Even J3
 U 1 1 62008AB1
 P 3050 3200
@@
 $EndComp
 $Comp
-L Connector_Generic:Conn_02x10_Counter_Clockwise J4
+L Connector_Generic:Conn_02x10_Odd_Even J4
 U 1 1 6200A2AB
 P 3850 3200
@@
 $EndComp
 $Comp
-L Connector_Generic:Conn_02x15_Counter_Clockwise J6
+L Connector_Generic:Conn_02x15_Odd_Even J6
 U 1 1 62019DEC
 P 6500 3400
@@
 $EndComp
 $Comp
-L Connector_Generic:Conn_02x15_Counter_Clockwise J7
+L Connector_Generic:Conn_02x15_Odd_Even J7
 U 1 1 6203836E
 P 7000 3400
@@
 	6300 4100 7300 4100
 $Comp
-L Connector_Generic:Conn_02x15_Counter_Clockwise J10
+L Connector_Generic:Conn_02x15_Odd_Even J10
 U 1 1 6204A5F5
 P 8100 3350
@@
 $EndComp
 $Comp
-L Connector_Generic:Conn_02x15_Counter_Clockwise J11
+L Connector_Generic:Conn_02x15_Odd_Even J11
 U 1 1 6204A5FB
 P 8600 3350
@@
 gpio 10
 $Comp
-L Connector_Generic:Conn_02x12_Counter_Clockwise J9
+L Connector_Generic:Conn_02x12_Odd_Even J9
 U 1 1 61FD1A5A
 P 7750 5350
