File: Boards/Main Board/RevB/Baja_Pi_Expansion/Baja_Pi_Expansion.kicad_pcb (KiCad board)
At the start: 2 copper layers, 85 x 56 mm, 20 parts, among them J1 Conn_02x10_Counter_Clockwise, J2 Conn_02x12_Counter_Clockwise, J3 Screw_Terminal_01x04, J4 Conn_02x20_Odd_Even, J5 Screw_Terminal_01x04, U1 HDSP-7403

Commit message: Fixed Main-RevB autorouting
Parts:
- removed G***: LOGO, Custom Footprints:RIT_Logo
Routing:
- net /gnd: track 0.00 -> 275.3 mm
- net /gpio8: track 0.00 -> 99.4 mm
- net /vcc: track 0.00 -> 98.7 mm, vias 0 -> 1
- net /gpio7: track 0.00 -> 96.0 mm
- net /reset: track 0.00 -> 92.9 mm
- net /gpio11: track 0.00 -> 91.6 mm, vias 0 -> 1
- net /gpio6: track 0.00 -> 91.3 mm, vias 0 -> 1
- net /5v: track 0.00 -> 77.3 mm
- net /gpio4: track 0.00 -> 67.9 mm
- net /gpio9: track 0.00 -> 63.9 mm, vias 0 -> 1
- net Net-(D1-Pad2): track 0.00 -> 59.9 mm
- net /gpio10: track 0.00 -> 58.3 mm
- net /gpio2: track 0.00 -> 57.5 mm
- net /gpio1: track 0.00 -> 57.3 mm
- net /3v3: track 0.00 -> 57.3 mm
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- removed copper zone on F.Cu, net /vcc
