File: Boards/Strain_Gauge_Schmatic/Strain_Guage_Schematic.sch (KiCad schematic (older format))
At the start: 16 parts, among them J1 Conn_01x03_Male, J2 Conn_01x02_Male, U1 LM358

Commit message: Added capacitor resistances
Parts:
- C5, C6, C7, C8, C9: value C -> 100nF
Changed lines of the file:
@@
 P 8375 3750
 F 0 "C6" H 8490 3796 50  0000 L CNN
-F 1 "C" H 8490 3705 50  0000 L CNN
+F 1 "100nF" H 8490 3705 50  0000 L CNN
 F 2 "Capacitor_SMD:C_0603_1608Metric" H 8413 3600 50  0001 C CNN
 F 3 "~" H 8375 3750 50  0001 C CNN
@@
 P 6850 2000
 F 0 "C7" H 6965 2046 50  0000 L CNN
-F 1 "C" H 6965 1955 50  0000 L CNN
+F 1 "100nF" H 6965 1955 50  0000 L CNN
 F 2 "Capacitor_SMD:C_0603_1608Metric" H 6888 1850 50  0001 C CNN
 F 3 "~" H 6850 2000 50  0001 C CNN
@@
 P 9400 2750
 F 0 "C8" H 9515 2796 50  0000 L CNN
-F 1 "C" H 9515 2705 50  0000 L CNN
+F 1 "100nF" H 9515 2705 50  0000 L CNN
 F 2 "Capacitor_SMD:C_0603_1608Metric" H 9438 2600 50  0001 C CNN
 F 3 "~" H 9400 2750 50  0001 C CNN
@@
 P 8350 1175
 F 0 "C9" H 8465 1221 50  0000 L CNN
-F 1 "C" H 8465 1130 50  0000 L CNN
+F 1 "100nF" H 8465 1130 50  0000 L CNN
 F 2 "Capacitor_SMD:C_0603_1608Metric" H 8388 1025 50  0001 C CNN
 F 3 "~" H 8350 1175 50  0001 C CNN
@@
 P 7575 2400
 F 0 "C5" H 7690 2446 50  0000 L CNN
-F 1 "C" H 7690 2355 50  0000 L CNN
+F 1 "100nF" H 7690 2355 50  0000 L CNN
 F 2 "Capacitor_SMD:C_0603_1608Metric" H 7613 2250 50  0001 C CNN
 F 3 "~" H 7575 2400 50  0001 C CNN
