File: Boards/Strain_Gauge_Schmatic/Regulator.sch (KiCad schematic (older format))
At the start: 5 parts

Commit message: Small error in strain gauge schematic, C4 footprint a bit big
Parts:
- C4: footprint Capacitor_Tantalum_SMD:CP_EIA-3216-18_Kemet-A -> Capacitor_SMD:C_0603_1608Metric
Changed lines of the file:
@@
 F 0 "C4" H 7568 2296 50  0000 L CNN
 F 1 "4.7uF_16V_cpu" H 7568 2205 50  0000 L CNN
-F 2 "Capacitor_Tantalum_SMD:CP_EIA-3216-18_Kemet-A" H 7488 2100 50  0001 C CNN
+F 2 "Capacitor_SMD:C_0603_1608Metric" H 7488 2100 50  0001 C CNN
 F 3 "~" H 7450 2250 50  0001 C CNN
 	1    7450 2250
