File: Boards/ADC Board/RevB/5v_regulator.sch (KiCad schematic (older format))
At the start: 7 parts

Commit message: Continued making RevB PCB
Parts:
- R9: value 350? -> 1.8k
Changed lines of the file:
@@
 AR Path="/61663709/61653277" Ref="R9"  Part="1"
 F 0 "R9" H 2618 2846 50  0000 L CNN
-F 1 "350?" H 2618 2755 50  0000 L CNN
+F 1 "1.8k" H 2618 2755 50  0000 L CNN
 F 2 "Resistor_SMD:R_0603_1608Metric" V 2590 2790 50  0001 C CNN
 F 3 "~" H 2550 2800 50  0001 C CNN
