File: Boards/ADC Board/RevB/RevA.sch (KiCad schematic (older format))
At the start: 6 parts, among them J1 Left Connector, J2 Right Connector, M2.5 CMH

Commit message: Began footprint associations for rev b
Parts:
- D2: renamed from D?; footprint (none) -> LED_SMD:LED_1206_3216Metric
- D3: renamed from D?; footprint (none) -> Diode_SMD:D_SMA
- gave numbers to parts that had none: 1
Changed lines of the file:
@@
 5V
 $Comp
-L Switch:SW_DIP_x01 SW?
+L Switch:SW_DIP_x01 SW1
 U 1 1 62322B6A
 P 3900 4500
-F 0 "SW?" H 3900 4767 50  0000 C CNN
+F 0 "SW1" H 3900 4767 50  0000 C CNN
 F 1 "SW_DIP_x01" H 3900 4676 50  0000 C CNN
 F 2 "" H 3900 4500 50  0001 C CNN
@@
 A7
 $Comp
-L Simulation_SPICE:DIODE D?
+L Simulation_SPICE:DIODE D3
 U 1 1 6232B450
 P 4050 1050
-F 0 "D?" H 4050 1267 50  0000 C CNN
+F 0 "D3" H 4050 1267 50  0000 C CNN
 F 1 "DIODE" H 4050 1176 50  0000 C CNN
-F 2 "" H 4050 1050 50  0001 C CNN
+F 2 "Diode_SMD:D_SMA" H 4050 1050 50  0001 C CNN
 F 3 "~" H 4050 1050 50  0001 C CNN
 F 4 "Y" H 4050 1050 50  0001 L CNN "Spice_Netlist_Enabled"
@@
 GND
 $Comp
-L Device:LED D?
+L Device:LED D2
 U 1 1 6233EF46
 P 3600 4650
-F 0 "D?" V 3639 4532 50  0000 R CNN
+F 0 "D2" V 3639 4532 50  0000 R CNN
 F 1 "LED" V 3548 4532 50  0000 R CNN
-F 2 "" H 3600 4650 50  0001 C CNN
+F 2 "LED_SMD:LED_1206_3216Metric" H 3600 4650 50  0001 C CNN
 F 3 "~" H 3600 4650 50  0001 C CNN
 	1    3600 4650

Commit message: Created PCB for Rev B
Parts:
- SW1: footprint (none) -> Button_Switch_SMD:SW_DIP_SPSTx01_Slide_9.78x4.72mm_W8.61mm_P2.54mm
Changed lines of the file:
@@
 F 0 "SW1" H 3900 4767 50  0000 C CNN
 F 1 "SW_DIP_x01" H 3900 4676 50  0000 C CNN
-F 2 "" H 3900 4500 50  0001 C CNN
+F 2 "Button_Switch_SMD:SW_DIP_SPSTx01_Slide_9.78x4.72mm_W8.61mm_P2.54mm" H 3900 4500 50  0001 C CNN
 F 3 "~" H 3900 4500 50  0001 C CNN
 	1    3900 4500

Commit message: Continued making RevB PCB
Parts:
- added R18: 1.8k, Resistor_SMD:R_0603_1608Metric, symbol Device:R_US
Connections:
- net 5V: now also R18.1; no longer D2.2 (A)
- new net: D2.2 (A), R18.2
Other:
- moved on the sheet: D2
Changed lines of the file:
@@
 Wire Wire Line
 	7100 3100 7250 3100
-Text Label 3400 4800 2    50   ~ 0
+Text Label 3400 5300 2    50   ~ 0
 GND
 $Comp
 L Device:LED D2
 U 1 1 6233EF46
-P 3600 4650
-F 0 "D2" V 3639 4532 50  0000 R CNN
-F 1 "LED" V 3548 4532 50  0000 R CNN
-F 2 "LED_SMD:LED_1206_3216Metric" H 3600 4650 50  0001 C CNN
-F 3 "~" H 3600 4650 50  0001 C CNN
-	1    3600 4650
+P 3600 5150
+F 0 "D2" V 3639 5032 50  0000 R CNN
+F 1 "LED" V 3548 5032 50  0000 R CNN
+F 2 "LED_SMD:LED_1206_3216Metric" H 3600 5150 50  0001 C CNN
+F 3 "~" H 3600 5150 50  0001 C CNN
+	1    3600 5150
 	0    -1   -1   0
 $EndComp
 Wire Wire Line
 	3400 4500 3600 4500
+Wire Wire Line
+	3400 5300 3600 5300
+$Comp
+L Device:R_US R18
+U 1 1 62356F25
+P 3600 4850
+AR Path="/62356F25" Ref="R18"  Part="1"
+AR Path="/6164E083/62356F25" Ref="R?"  Part="1"
+AR Path="/61663709/62356F25" Ref="R?"  Part="1"
+F 0 "R18" H 3668 4896 50  0000 L CNN
+F 1 "1.8k" H 3668 4805 50  0000 L CNN
+F 2 "Resistor_SMD:R_0603_1608Metric" V 3640 4840 50  0001 C CNN
+F 3 "~" H 3600 4850 50  0001 C CNN
+	1    3600 4850
+	1    0    0    -1
+$EndComp
+Wire Wire Line
+	3600 4700 3600 4500
 Connection ~ 3600 4500
-Wire Wire Line
-	3400 4800 3600 4800
 $EndSCHEMATC
