File: Boards/ADC Board/RevB/controller.sch (KiCad schematic (older format))
At the start: 4 parts

Commit message: Began footprint associations for rev b
Parts:
- C5: renamed from C?; footprint (none) -> Capacitor_SMD:C_0603_1608Metric
- J21: renamed from J?; footprint (none) -> Connector_PinHeader_2.54mm:PinHeader_2x03_P2.54mm_Vertical
- U1: renamed from U?; footprint 32M1-A_ATM -> (none)
- Y1: renamed from Y?; footprint OSC_CSTCE16M0V53-R0 -> (none)
Changed lines of the file:
@@
 $EndDescr
 $Comp
-L CSTCE16M0V53-R0:CSTCE16M0V53-R0 Y?
+L CSTCE16M0V53-R0:CSTCE16M0V53-R0 Y1
 U 1 1 6234D0B2
 P 1600 4450
-F 0 "Y?" H 1600 4817 50  0000 C CNN
+F 0 "Y1" H 1600 4817 50  0000 C CNN
 F 1 "CSTCE16M0V53-R0" H 1600 4726 50  0000 C CNN
-F 2 "OSC_CSTCE16M0V53-R0" H 1600 4450 50  0001 L BNN
+F 2 "" H 1600 4450 50  0001 L BNN
 F 3 "1.0 mm" H 1600 4450 50  0001 L BNN
 F 4 "Murata Electronics" H 1600 4450 50  0001 L BNN "Field4"
@@
 	9100 4900 9250 4900
 $Comp
-L Device:C C?
+L Device:C C5
 U 1 1 6235B1D1
 P 8650 4950
-F 0 "C?" V 8398 4950 50  0000 C CNN
+F 0 "C5" V 8398 4950 50  0000 C CNN
 F 1 "100nF" V 8489 4950 50  0000 C CNN
-F 2 "" H 8688 4800 50  0001 C CNN
+F 2 "Capacitor_SMD:C_0603_1608Metric" H 8688 4800 50  0001 C CNN
 F 3 "~" H 8650 4950 50  0001 C CNN
 	1    8650 4950
@@
 NoConn ~ 2900 5050
 $Comp
-L 2020-11-11_15-40-12:ATMEGA328P-MUR U?
+L 2020-11-11_15-40-12:ATMEGA328P-MUR U1
 U 1 1 6234A28C
 P 2900 3750
-F 0 "U?" H 5700 4137 60  0000 C CNN
+F 0 "U1" H 5700 4137 60  0000 C CNN
 F 1 "ATMEGA328P-MUR" H 5700 4031 60  0000 C CNN
-F 2 "32M1-A_ATM" H 5700 3990 60  0001 C CNN
+F 2 "" H 5700 3990 60  0001 C CNN
 F 3 "" H 2900 3750 60  0000 C CNN
 	1    2900 3750
@@
 D3
 $Comp
-L Connector_Generic:Conn_02x03_Odd_Even J?
+L Connector_Generic:Conn_02x03_Odd_Even J21
 U 1 1 62316B37
 P 1500 5900
-F 0 "J?" H 1550 6217 50  0000 C CNN
+F 0 "J21" H 1550 6217 50  0000 C CNN
 F 1 "Conn_02x03_Odd_Even" H 1550 6126 50  0000 C CNN
-F 2 "" H 1500 5900 50  0001 C CNN
+F 2 "Connector_PinHeader_2.54mm:PinHeader_2x03_P2.54mm_Vertical" H 1500 5900 50  0001 C CNN
 F 3 "~" H 1500 5900 50  0001 C CNN
 	1    1500 5900

Commit message: Created PCB for Rev B
Parts:
- U1: footprint (none) -> ATMEGA_Import:ATMEGA328P-MUR
- Y1: footprint (none) -> CSTCE16M0V53-R0:OSC_CSTCE16M0V53-R0
Changed lines of the file:
@@
 F 0 "Y1" H 1600 4817 50  0000 C CNN
 F 1 "CSTCE16M0V53-R0" H 1600 4726 50  0000 C CNN
-F 2 "" H 1600 4450 50  0001 L BNN
+F 2 "CSTCE16M0V53-R0:OSC_CSTCE16M0V53-R0" H 1600 4450 50  0001 L BNN
 F 3 "1.0 mm" H 1600 4450 50  0001 L BNN
 F 4 "Murata Electronics" H 1600 4450 50  0001 L BNN "Field4"
@@
 F 0 "U1" H 5700 4137 60  0000 C CNN
 F 1 "ATMEGA328P-MUR" H 5700 4031 60  0000 C CNN
-F 2 "" H 5700 3990 60  0001 C CNN
+F 2 "ATMEGA_Import:ATMEGA328P-MUR" H 5700 3990 60  0001 C CNN
 F 3 "" H 2900 3750 60  0000 C CNN
 	1    2900 3750

Commit message: Continued making RevB PCB
Parts:
- U1: footprint ATMEGA_Import:ATMEGA328P-MUR -> ATMEGA:ATMEGA328P-MUR
Changed lines of the file:
@@
 F 0 "U1" H 5700 4137 60  0000 C CNN
 F 1 "ATMEGA328P-MUR" H 5700 4031 60  0000 C CNN
-F 2 "ATMEGA_Import:ATMEGA328P-MUR" H 5700 3990 60  0001 C CNN
+F 2 "ATMEGA:ATMEGA328P-MUR" H 5700 3990 60  0001 C CNN
 F 3 "" H 2900 3750 60  0000 C CNN
 	1    2900 3750
