File: Boards/ADC Board/RevB/RevA.kicad_pcb (KiCad board)
At the start: 2 copper layers, 85 x 56 mm, 31 parts, among them J1 Left Connector, J10 Jumper Terminals, J11 Arduino Nano L, J12 Arduino Nano R, J13 Extra Pins, J14 Screw Terminals, J16 Screw Terminals, J2 Right Connector, J3 Screw Terminals, J4 Jumper Terminals, J5 Screw Terminals, J6 Jumper Terminals, J7 Screw Terminals, J8 Jumper Terminals, J9 Screw Terminals, M2.5 CMH

Commit message: Cleanup before pcb
Parts:
- removed J10, J4, J6, J8: Jumper Terminals, Connector_PinHeader_2.54mm:PinHeader_1x03_P2.54mm_Vertical
- removed J11: Arduino Nano L, Connector_PinSocket_2.54mm:PinSocket_1x15_P2.54mm_Vertical
- removed J12: Arduino Nano R, Connector_PinSocket_2.54mm:PinSocket_1x15_P2.54mm_Vertical
- removed J13: Extra Pins, Connector_PinHeader_2.54mm:PinHeader_2x03_P2.54mm_Vertical
- removed J14, J16, J3, J5, J7, J9: Screw Terminals, Spring_Terminal_4Pin:1984989
- removed R1, R2, R3, R4, R5, R6, R7, R8: 10k, Resistor_SMD:R_0603_1608Metric
Routing:
- net /5V: track 242.6 -> 0.00 mm
- net /I2C_Data: track 82.2 -> 0.00 mm
- net /I2C_Clock: track 76.8 -> 0.00 mm
- net /Analog_0: track 72.5 -> 0.00 mm
- net /Digital_0: track 68.3 -> 0.00 mm
- net /Digital_1: track 61.7 -> 0.00 mm
- net /Analog_1: track 59.6 -> 0.00 mm
- net /Digital_2: track 57.7 -> 0.00 mm
- net /Digital_3: track 49.5 -> 0.00 mm
- net /Analog_2: track 49.3 -> 0.00 mm
- net /Reset: track 45.0 -> 0.00 mm
- net /Analog_3: track 38.0 -> 0.00 mm
- net /VCC: track 37.0 -> 0.00 mm
- net /3.3V: track 21.7 -> 0.00 mm
- net /Controller/D12: track 21.2 -> 0.00 mm
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Other:
- board text removed: "5V"
- board text removed: "5V A0 GND 5V"
- board text removed: "5V D0 GND 5V"
- board text removed: "A0"
- board text removed: "A1"
- board text removed: "A1 GND 5V A2"
- board text removed: "A2"
- board text removed: "A3"
- board text removed: "Analog Pins"
- board text removed: "D0"
- board text removed: "D1"
- board text removed: "D1 GND 5V D2"
- board text removed: "D2"
- board text removed: "D3"
- board text removed: "Digital Pins"
- board text removed: "GND"
- board text removed: "GND 5V A3 GND"
- board text removed: "GND 5V D3 GND"
- board text removed: "JLCJLCJLCJLC"
- board text removed: "SDAQ ADC Board Revision A Chris Walters (508) 975-3337 RIT BAJA"

Commit message: Created PCB for Rev B
Parts:
- added C5: 100nF, Capacitor_SMD:C_0603_1608Metric, F.Cu at (148.5, 34.0)
- added D2: LED, LED_SMD:LED_1206_3216Metric, F.Cu at (80.3, 73.4)
- added D3: DIODE, Diode_SMD:D_SMA, F.Cu at (68.8, 80.5)
- added J10: Screw_Terminal_01x04, Spring_Terminal_4Pin:1984989, F.Cu at (87.0, 40.9)
- added J11: Screw_Terminal_01x04, Spring_Terminal_4Pin:1984989, F.Cu at (69.0, 54.4)
- added J12: Conn_02x05_Top_Bottom, Connector_PinHeader_2.54mm:PinHeader_2x05_P2.54mm_Vertical, F.Cu at (121.0, 35.1)
- added J13: Conn_01x03_Male, Connector_PinHeader_2.54mm:PinHeader_1x03_P2.54mm_Vertical, F.Cu at (67.1, 88.8)
- added J14: Conn_01x03_Male, Connector_PinHeader_2.54mm:PinHeader_1x03_P2.54mm_Vertical, F.Cu at (134.0, 49.4)
- added J15: Conn_01x03_Male, Connector_PinHeader_2.54mm:PinHeader_1x03_P2.54mm_Vertical, F.Cu at (87.5, 88.8)
- added J16: Conn_01x03_Male, Connector_PinHeader_2.54mm:PinHeader_1x03_P2.54mm_Vertical, F.Cu at (157.1, 35.1)
- added J17: Conn_01x03_Male, Connector_PinHeader_2.54mm:PinHeader_1x03_P2.54mm_Vertical, F.Cu at (111.5, 74.1)
- added J18: Conn_01x03_Male, Connector_PinHeader_2.54mm:PinHeader_1x03_P2.54mm_Vertical, F.Cu at (134.0, 62.2)
- added J19: Conn_01x03_Male, Connector_PinHeader_2.54mm:PinHeader_1x03_P2.54mm_Vertical, F.Cu at (154.4, 49.4)
- added J20: Conn_01x03_Male, Connector_PinHeader_2.54mm:PinHeader_1x03_P2.54mm_Vertical, F.Cu at (111.5, 86.8)
- added J21: Conn_02x03_Odd_Even, Connector_PinHeader_2.54mm:PinHeader_2x03_P2.54mm_Vertical, F.Cu at (134.0, 35.1)
- added J22: Conn_01x03_Female, Connector_PinHeader_1.27mm:PinHeader_1x03_P1.27mm_Vertical, F.Cu at (103.1, 73.4)
- added J3: Conn_01x03_Female, Connector_PinHeader_1.27mm:PinHeader_1x03_P1.27mm_Vertical, F.Cu at (90.7, 73.4)
- added J4: Conn_01x03_Female, Connector_PinHeader_1.27mm:PinHeader_1x03_P1.27mm_Vertical, F.Cu at (94.8, 73.4)
- added J5: Conn_01x03_Female, Connector_PinHeader_1.27mm:PinHeader_1x03_P1.27mm_Vertical, F.Cu at (99.0, 73.4)
- added J6: Screw_Terminal_01x04, Spring_Terminal_4Pin:1984989, F.Cu at (104.9, 54.4)
- added J7: Screw_Terminal_01x04, Spring_Terminal_4Pin:1984989, F.Cu at (104.9, 40.9)
- added J8: Screw_Terminal_01x04, Spring_Terminal_4Pin:1984989, F.Cu at (87.0, 54.4)
- added J9: Screw_Terminal_01x04, Spring_Terminal_4Pin:1984989, F.Cu at (69.0, 40.9)
- added R1: 10k, Resistor_SMD:R_0603_1608Metric, F.Cu at (71.4, 87.7)
- added R10: 10k, Resistor_SMD:R_0603_1608Metric, F.Cu at (115.8, 73.0)
- added R11: 10k, Resistor_SMD:R_0603_1608Metric, F.Cu at (119.8, 73.0)
- added R12: 10k, Resistor_SMD:R_0603_1608Metric, F.Cu at (138.4, 61.1)
- added R13: 10k, Resistor_SMD:R_0603_1608Metric, F.Cu at (142.4, 61.1)
- added R14: 10k, Resistor_SMD:R_0603_1608Metric, F.Cu at (158.7, 48.3)
- added R15: 10k, Resistor_SMD:R_0603_1608Metric, F.Cu at (162.7, 48.3)
- added R16: 10k, Resistor_SMD:R_0603_1608Metric, F.Cu at (115.8, 85.8)
- added R17: 10k, Resistor_SMD:R_0603_1608Metric, F.Cu at (119.8, 85.8)
- added R2: 10k, Resistor_SMD:R_0603_1608Metric, F.Cu at (75.4, 87.7)
- added R3: 10k, Resistor_SMD:R_0603_1608Metric, F.Cu at (138.4, 48.3)
- added R4: 10k, Resistor_SMD:R_0603_1608Metric, F.Cu at (142.4, 48.3)
- added R5: 10k, Resistor_SMD:R_0603_1608Metric, F.Cu at (91.8, 87.7)
- added R6: 10k, Resistor_SMD:R_0603_1608Metric, F.Cu at (95.8, 87.7)
- added R7: 10k, Resistor_SMD:R_0603_1608Metric, F.Cu at (165.5, 34.0)
- added R8: 10k, Resistor_SMD:R_0603_1608Metric, F.Cu at (161.5, 34.0)
- added SW1: SW_DIP_x01, Button_Switch_SMD:SW_DIP_SPSTx01_Slide_9.78x4.72mm_W8.61mm_P2.54mm, F.Cu at (71.1, 75.0)
- added Y1: CSTCE16M0V53-R0, CSTCE16M0V53-R0:OSC_CSTCE16M0V53-R0, F.Cu at (141.3, 42.2)
Connections:
- net /5V renamed /5v_regulator/5V
- J2 pad 22: /Reset -> Net-(D3-Pad1)

Commit message: Continued making RevB PCB
Parts:
- added R18: 1.8k, Resistor_SMD:R_0603_1608Metric, F.Cu at (234.9, 105.9)
- added U1: ATMEGA328P-MUR, ATMEGA:ATMEGA328P-MUR, F.Cu at (225.8, 81.0)
- R9: value 350? -> 1.8k
- moved D3 165.1 mm to (233.7, 88.1)
- moved D2 154.0 mm to (230.1, 109.0)
- moved SW1 154.0 mm to (221.0, 110.5)
- moved J11 146.7 mm to (199.9, 120.7)
- moved J3 133.0 mm to (221.7, 96.0)
- moved J5 133.0 mm to (230.0, 96.0)
- moved J22 133.0 mm to (234.2, 96.0)
- moved J4 132.4 mm to (225.3, 96.0)
- moved J9 125.3 mm to (165.6, 120.7)
- moved J10 124.6 mm to (182.6, 120.7)
- moved J8 123.7 mm to (208.8, 75.7), turned to 180 degrees
- moved C5 94.7 mm to (230.6, 81.3), turned to 90 degrees
- moved J7 93.8 mm to (192.0, 75.7), turned to 180 degrees
- moved Y1 88.8 mm to (221.0, 81.3), turned to 90 degrees
- moved J6 73.3 mm to (175.1, 75.7), turned to 180 degrees
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Connections:
- D2 pad 2: /5V -> Net-(D2-Pad2)

Commit message: Completed placements on RevB, prepared for auto routing.
Parts:
- moved J21 135.0 mm to (236.1, 123.5), turned to 90 degrees
- moved J12 117.2 mm to (231.0, 75.6), turned to 90 degrees
- moved A0 104.5 mm to (171.5, 92.8)
- moved R1 104.5 mm to (171.5, 100.8)
- moved R2 104.5 mm to (171.5, 102.8)
- moved R17 102.1 mm to (210.1, 94.5), turned to 180 degrees
- moved D1 102.0 mm to (210.1, 104.8), turned to 180 degrees
- moved R16 101.6 mm to (210.1, 96.5), turned to 180 degrees
- moved A2 92.1 mm to (179.5, 92.8)
- moved R5 92.1 mm to (179.5, 100.8)
- moved R6 92.1 mm to (179.5, 102.8)
- moved D0 80.7 mm to (214.1, 104.8), turned to 180 degrees
- moved R10 78.4 mm to (187.5, 100.8)
- moved R11 78.4 mm to (187.5, 102.8)
- moved A4 78.3 mm to (187.5, 92.8)
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- renumbered J13 to A0, J14 to A1, J15 to A2, J16 to A3, J17 to A4, J18 to A5, J19 to D0, J20 to D1
Other:
- board text added: "0x 0 0 0 0"
- board text added: "0x 1 1 1 1"
- board text added: "5V"
- board text added: "5V A4 GND 5V"
- board text added: "5V GND A0 5V"
- board text added: "A0"
- board text added: "A1"
- board text added: "A2"
- board text added: "A2 5V GND A1"
- board text added: "A3"
- board text added: "A4"
- board text added: "A5"
- board text added: "A5 GND 5V D0"
- board text added: "Board ID"
- board text added: "D0"
- board text added: "D1"
- board text added: "Expansion Port"
- board text added: "GND"
- board text added: "GND 5V D1 GND"
- board text added: "GND A3 5V GND"
- board text added: "JLCJLCJLCJLC"
- board text added: "Programming Port"
- board text added: "Pull-down"
- board text added: "Pull-up"
- board text added: "SDAQ ADC Board Revision B Chris Walters (508) 975-3337 RIT BAJA"

Commit message: Completed RevB autorouting
Parts:
- moved J22 9.62 mm to (222.8, 91.7)
- moved J3 5.62 mm to (230.4, 91.7)
- moved J5 4.54 mm to (225.3, 91.7)
- moved J4 0.54 mm to (227.9, 91.7)
- moved C5 0.50 mm to (229.1, 111.9)
- moved Y1 0.50 mm to (219.5, 111.9)
- moved C1 0.50 mm to (233.5, 82.6)
- moved C2 0.50 mm to (221.0, 79.7)
- moved C3 0.50 mm to (221.0, 85.7)
- moved C4 0.50 mm to (220.0, 82.7)
- moved VR1 0.50 mm to (228.0, 82.7)
- moved U1 0.50 mm to (224.6, 111.7)
- renumbered A0 to J13, A1 to J14, A2 to J15, A3 to J16, A4 to J17, A5 to J18, D0 to J19, D1 to J20
Routing:
- net /5V: track 0.00 -> 310.0 mm, vias 0 -> 2
- net /A4: track 0.00 -> 141.5 mm, vias 0 -> 2
- net /A3: track 0.00 -> 137.0 mm, vias 0 -> 1
- net /A5: track 0.00 -> 125.8 mm, vias 0 -> 1
- net /A0: track 0.00 -> 117.5 mm, vias 0 -> 1
- net /A2: track 0.00 -> 115.9 mm, vias 0 -> 1
- net /A1: track 0.00 -> 113.0 mm, vias 0 -> 1
- net /A6: track 0.00 -> 97.8 mm, vias 0 -> 1
- net /A7: track 0.00 -> 84.8 mm, vias 0 -> 1
- net /I2C_Data: track 0.00 -> 73.3 mm, vias 0 -> 1
- net /I2C_Clock: track 0.00 -> 70.0 mm, vias 0 -> 1
- net /5v_regulator/5V: track 0.00 -> 58.8 mm, vias 0 -> 2
- net /VCC: track 0.00 -> 54.1 mm, vias 0 -> 1
- net /Reset: track 0.00 -> 35.7 mm, vias 0 -> 1
- net /GND: track 0.00 -> 25.8 mm, vias 0 -> 6
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Other:
- copper layers 2 -> 4
- board text added: "A0 A1 A2 A3 A4 A5"
- board text added: "D1 D0"
