File: Boards/Brakes Relay Board/RevA/relay_board.kicad_sch (KiCad schematic)
At the start: 15 parts

Commit message: Prepared RevA Relay Board PCB
Parts:
- D1: renamed from D?; value (none) -> LED
- J1: renamed from J?; value (none) -> Screw_Terminal_01x04
- R1: renamed from R?; value (none) -> R
- U1: renamed from U?; value (none) -> ALQ105
- U2, U3, U4, U5, U6: renamed from U?; footprint PAN_ALQ1_PAN -> (none)
- gave numbers to parts that had none: 6
Other:
- moved on the sheet: U6

Commit message: updated LED resistor on relay board rev A
Parts:
- D1: footprint (none) -> Diode_SMD:D_1206_3216Metric
- J1, J2, J3, J4, J7: footprint (none) -> BAJA-4PIN:1984989
- J5: footprint (none) -> Connector_PinHeader_2.54mm:PinHeader_2x10_P2.54mm_Vertical
- J6: footprint (none) -> Connector_PinHeader_2.54mm:PinHeader_2x12_P2.54mm_Vertical
- R1: value R -> (none); footprint (none) -> Resistor_SMD:R_0603_1608Metric
- U1, U2, U3, U4, U5, U6: footprint (none) -> ALQ105-BAJA-FP:ALQ105
Changed lines of the file:
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@@
       (effects (font (size 1.524 1.524)))
     )
-    (property "Footprint" "" (id 2) (at 255.27 15.494 0)
+    (property "Footprint" "ALQ105-BAJA-FP:ALQ105" (id 2) (at 255.27 15.494 0)
       (effects (font (size 1.524 1.524)) hide)
     )
@@
       (effects (font (size 1.524 1.524)))
     )
-    (property "Footprint" "" (id 2) (at 255.905 64.389 0)
+    (property "Footprint" "ALQ105-BAJA-FP:ALQ105" (id 2) (at 255.905 64.389 0)
       (effects (font (size 1.524 1.524)) hide)
     )
@@
       (effects (font (size 1.27 1.27)) (justify left))
     )
-    (property "Footprint" "" (id 2) (at 33.655 137.16 0)
+    (property "Footprint" "BAJA-4PIN:1984989" (id 2) (at 33.655 137.16 0)
       (effects (font (size 1.27 1.27)) hide)
     )
@@
       (effects (font (size 1.27 1.27)) (justify right))
     )
-    (property "Footprint" "" (id 2) (at 80.645 97.79 0)
+    (property "Footprint" "Diode_SMD:D_1206_3216Metric" (id 2) (at 80.645 97.79 0)
       (effects (font (size 1.27 1.27)) hide)
     )
@@
       (effects (font (size 1.27 1.27)) (justify left))
     )
-    (property "Footprint" "" (id 2) (at 33.655 120.015 0)
+    (property "Footprint" "BAJA-4PIN:1984989" (id 2) (at 33.655 120.015 0)
       (effects (font (size 1.27 1.27)) hide)
     )
@@
       (effects (font (size 1.524 1.524)))
     )
-    (property "Footprint" "" (id 2) (at 142.24 65.024 0)
+    (property "Footprint" "ALQ105-BAJA-FP:ALQ105" (id 2) (at 142.24 65.024 0)
       (effects (font (size 1.524 1.524)) hide)
     )
@@
       (effects (font (size 1.27 1.27)) (justify left))
     )
-    (property "Value" "R" (id 1) (at 82.55 91.4399 0)
-      (effects (font (size 1.27 1.27)) (justify left))
-    )
-    (property "Footprint" "" (id 2) (at 78.867 90.17 90)
+    (property "Value" "" (id 1) (at 82.55 91.4399 0)
+      (effects (font (size 1.27 1.27)) (justify left))
+    )
+    (property "Footprint" "Resistor_SMD:R_0603_1608Metric" (id 2) (at 78.867 90.17 90)
       (effects (font (size 1.27 1.27)) hide)
     )
@@
       (effects (font (size 1.524 1.524)))
     )
-    (property "Footprint" "" (id 2) (at 199.39 16.764 0)
+    (property "Footprint" "ALQ105-BAJA-FP:ALQ105" (id 2) (at 199.39 16.764 0)
       (effects (font (size 1.524 1.524)) hide)
     )
@@
       (effects (font (size 1.27 1.27)) (justify left))
     )
-    (property "Footprint" "" (id 2) (at 33.655 150.495 0)
+    (property "Footprint" "BAJA-4PIN:1984989" (id 2) (at 33.655 150.495 0)
       (effects (font (size 1.27 1.27)) hide)
     )
@@
       (effects (font (size 1.27 1.27)) (justify left))
     )
-    (property "Footprint" "" (id 2) (at 34.925 167.005 0)
+    (property "Footprint" "BAJA-4PIN:1984989" (id 2) (at 34.925 167.005 0)
       (effects (font (size 1.27 1.27)) hide)
     )
@@
       (effects (font (size 1.524 1.524)))
     )
-    (property "Footprint" "" (id 2) (at 199.39 65.024 0)
+    (property "Footprint" "ALQ105-BAJA-FP:ALQ105" (id 2) (at 199.39 65.024 0)
       (effects (font (size 1.524 1.524)) hide)
     )
@@
     (property "Reference" "J5" (id 0) (at 44.45 20.32 0))
     (property "Value" "Conn_02x10_Counter_Clockwise" (id 1) (at 44.45 22.86 0))
-    (property "Footprint" "" (id 2) (at 43.18 36.83 0)
+    (property "Footprint" "Connector_PinHeader_2.54mm:PinHeader_2x10_P2.54mm_Vertical" (id 2) (at 43.18 36.83 0)
       (effects (font (size 1.27 1.27)) hide)
     )
@@
     (property "Reference" "J6" (id 0) (at 77.47 16.51 0))
     (property "Value" "Conn_02x12_Counter_Clockwise" (id 1) (at 77.47 19.05 0))
-    (property "Footprint" "" (id 2) (at 76.2 35.56 0)
+    (property "Footprint" "Connector_PinHeader_2.54mm:PinHeader_2x12_P2.54mm_Vertical" (id 2) (at 76.2 35.56 0)
       (effects (font (size 1.27 1.27)) hide)
     )
@@
       (effects (font (size 1.524 1.524)))
     )
-    (property "Footprint" "" (id 2) (at 142.24 16.764 0)
+    (property "Footprint" "ALQ105-BAJA-FP:ALQ105" (id 2) (at 142.24 16.764 0)
       (effects (font (size 1.524 1.524)) hide)
     )
@@
       (effects (font (size 1.27 1.27)) (justify left))
     )
-    (property "Footprint" "" (id 2) (at 116.84 136.525 0)
+    (property "Footprint" "BAJA-4PIN:1984989" (id 2) (at 116.84 136.525 0)
       (effects (font (size 1.27 1.27)) hide)
     )
@@
     )
     (path "/2e7a0426-12c9-4aa5-92b6-63a77b09669e"
-      (reference "R1") (unit 1) (value "R") (footprint "Resistor_SMD:R_0603_1608Metric")
+      (reference "R1") (unit 1) (value "1800") (footprint "Resistor_SMD:R_0603_1608Metric")
     )
     (path "/f862dac0-de9d-42c5-b0b0-17c723e7dfb0"
