File: Boards/Main Board/RevD/Baja_Pi_Expansion/Baja_Pi_Expansion.kicad_pcb (KiCad board)
At the start: 2 copper layers, 85 x 56 mm, 21 parts, among them J1 Conn_02x10_Counter_Clockwise, J2 Conn_02x12_Counter_Clockwise, J3 Screw_Terminal_01x04, J4 Conn_02x20_Odd_Even, J5 Screw_Terminal_01x04, J6 poe_choice, J7 rpi_poe_header

Commit message: Adding tons of random parsing scripts
(Needs cleanup)
Other:
- board text removed: "JLCJLCJLCJLC"
