File: Boards/Brakes Relay Board/RevB/5v_regulator.kicad_sch (KiCad schematic)
At the start: 5 parts

Commit message: Added new components to PCB
Parts:
- C1, C2, C3: value (none) -> ~; footprint (none) -> Capacitor_SMD:C_0603_1608Metric
- C4: value (none) -> ~; footprint (none) -> Capacitor_SMD:C_1206_3216Metric
- VR1: value (none) -> ~
Changed lines of the file:
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@@
       (effects (font (size 1.27 1.27)) (justify left))
     )
-    (property "Value" "" (id 1) (at 99.441 59.563 0)
+    (property "Value" "~" (id 1) (at 99.441 59.563 0)
       (effects (font (size 1.27 1.27)) (justify left))
     )
-    (property "Footprint" "" (id 2) (at 97.4852 62.23 0)
+    (property "Footprint" "Capacitor_SMD:C_0603_1608Metric" (id 2) (at 97.4852 62.23 0)
       (effects (font (size 1.27 1.27)) hide)
     )
@@
       (effects (font (size 1.27 1.27)) (justify left))
     )
-    (property "Value" "" (id 1) (at 154.051 57.023 0)
+    (property "Value" "~" (id 1) (at 154.051 57.023 0)
       (effects (font (size 1.27 1.27)) (justify left))
     )
-    (property "Footprint" "" (id 2) (at 152.0952 59.69 0)
+    (property "Footprint" "Capacitor_SMD:C_0603_1608Metric" (id 2) (at 152.0952 59.69 0)
       (effects (font (size 1.27 1.27)) hide)
     )
@@
       (effects (font (size 1.27 1.27)) (justify left))
     )
-    (property "Value" "" (id 1) (at 175.641 58.293 0)
+    (property "Value" "~" (id 1) (at 175.641 58.293 0)
       (effects (font (size 1.27 1.27)) (justify left))
     )
-    (property "Footprint" "" (id 2) (at 173.6852 60.96 0)
+    (property "Footprint" "Capacitor_SMD:C_0603_1608Metric" (id 2) (at 173.6852 60.96 0)
       (effects (font (size 1.27 1.27)) hide)
     )
@@
       (effects (font (size 1.27 1.27)) (justify left))
     )
-    (property "Value" "" (id 1) (at 192.2272 58.293 0)
+    (property "Value" "~" (id 1) (at 192.2272 58.293 0)
       (effects (font (size 1.27 1.27)) (justify left))
     )
-    (property "Footprint" "" (id 2) (at 190.1952 60.96 0)
+    (property "Footprint" "Capacitor_SMD:C_1206_3216Metric" (id 2) (at 190.1952 60.96 0)
       (effects (font (size 1.27 1.27)) hide)
     )
@@
     (in_bom yes) (on_board yes)
     (property "Reference" "VR1" (id 0) (at 125.73 44.0182 0))
-    (property "Value" "" (id 1) (at 125.73 46.3296 0))
+    (property "Value" "~" (id 1) (at 125.73 46.3296 0))
     (property "Footprint" "" (id 2) (at 125.73 53.34 0)
       (effects (font (size 1.27 1.27)) (justify left bottom) hide)
