File: Boards/Brakes Relay Board/RevB/relay_new.kicad_sch (KiCad schematic)
At the start: 5 parts, among them U1 ALQ105

Commit message: Added new components to PCB
Parts:
- D2: footprint (none) -> Diode_SMD:D_SMA
- MOSFET1: footprint TO252_AOS -> (none)
- R2, R3: footprint (none) -> Resistor_SMD:R_0603_1608Metric
- U1: footprint PAN_ALQ1_PAN -> (none)
Changed lines of the file:
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@@
       (effects (font (size 1.27 1.27)) (justify left))
     )
-    (property "Footprint" "" (id 2) (at 75.946 114.554 90)
+    (property "Footprint" "Resistor_SMD:R_0603_1608Metric" (id 2) (at 75.946 114.554 90)
       (effects (font (size 1.27 1.27)) hide)
     )
@@
       (effects (font (size 1.524 1.524)))
     )
-    (property "Footprint" "PAN_ALQ1_PAN" (id 2) (at 136.525 59.309 0)
+    (property "Footprint" "" (id 2) (at 136.525 59.309 0)
       (effects (font (size 1.524 1.524)) hide)
     )
@@
       (effects (font (size 1.524 1.524)) (justify left))
     )
-    (property "Footprint" "TO252_AOS" (id 2) (at 94.615 115.189 0)
+    (property "Footprint" "" (id 2) (at 94.615 115.189 0)
       (effects (font (size 1.524 1.524)) hide)
     )
@@
     (property "Reference" "R2" (id 0) (at 67.945 102.87 90))
     (property "Value" "100" (id 1) (at 67.945 105.41 90))
-    (property "Footprint" "" (id 2) (at 67.691 109.601 90)
+    (property "Footprint" "Resistor_SMD:R_0603_1608Metric" (id 2) (at 67.691 109.601 90)
       (effects (font (size 1.27 1.27)) hide)
     )
@@
       (effects (font (size 1.27 1.27)) (justify right))
     )
-    (property "Footprint" "" (id 2) (at 90.805 89.535 0)
+    (property "Footprint" "Diode_SMD:D_SMA" (id 2) (at 90.805 89.535 0)
       (effects (font (size 1.27 1.27)) hide)
     )
