File: Boards/Neo_Strain_Gauge/Strain_Gauge/Strain_Gauge.kicad_sch (KiCad schematic)
At the start: 58 parts, among them J1 Screw_Terminal_01x03, J2 Screw_Terminal_01x03, J3 Screw_Terminal_01x03, J4 Screw_Terminal_01x03, J5 Conn_01x02, J6 USB_B_Micro, J7 Conn_02x10_Counter_Clockwise, J8 Conn_02x12_Counter_Clockwise, U1 W25Q128JVS, U2 NCP1117-3.3_SOT223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

Commit message: More strain gauge work to get in-stock parts
Parts:
- removed U6: KA78M05_TO252, Package_TO_SOT_SMD:TO-252-2, symbol Regulator_Linear:KA78M05_TO252
- added C22: 10u, Capacitor_SMD:C_0603_1608Metric, symbol Device:C
- added U6: AZ1117-5.0, Package_TO_SOT_SMD:SOT-223-3_TabPin2, symbol Regulator_Linear:AZ1117-5.0
- C11, C12, C13, C14, C15, C16, C6, C7, C9: Purchase Link (none) -> https://www.digikey.com/en/products/detail/kyocera-avx/0402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
- C20: value 10u -> 22u
- C21, C3: footprint Capacitor_SMD:C_0603_1608Metric -> Capacitor_SMD:C_0402_1005Metric; Purchase Link (none) -> https://www.digikey.com/en/products/detail/kyocera-avx/0402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
- D1: Purchase Link (none) -> https://www.digikey.com/en/products/detail/diodes-incorpora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
- J6: Purchase Link (none) -> https://www.digikey.com/en/products/detail/amphenol-cs-fci/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
- U5: Purchase Link (none) -> https://www.digikey.com/en/products/detail/texas-instrument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
- Y1: Purchase Link (none) -> https://www.digikey.com/en/products/detail/abracon-llc/ABLS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
Connections:
- net +5V: now also U6.2 (VO)
- net GND: now also C22.2, U6.1 (GND)
- net rpi_5v: now also C22.1, U6.3 (VI)
- net VBUS: now reaches D1.1, J6.1 (VBUS)
- net REG_POWER: now reaches C4.1, D1.3, U2.3 (VI)

Commit message: Improve differential pairing.
Connections:
- net IN1+: now reaches R10.1, R9.2, U3.6 (IN1+)
- net IN3+: now reaches R5.2, R6.1, U3.2 (IN3+)
- net IN0+: now reaches R11.2, R12.1, U3.8 (IN0+)
- net IN3-: now reaches J1.2 (Pin_2), U3.1 (IN3-)
- net IN2-: now reaches J2.2 (Pin_2), U3.3 (IN2-)
- net IN2+: now reaches R7.2, R8.1, U3.4 (IN2+)
- net IN1-: now reaches J3.2 (Pin_2), U3.5 (IN1-)
- net IN0-: now reaches J4.2 (Pin_2), U3.7 (IN0-)
