File: Boards/Neo_Strain_Gauge/Strain_Gauge_V2/RPi.kicad_sch (KiCad schematic)
At the start: 31 parts, among them J5 Conn_01x02, SW1 SW_DIP_x04, U1 W25Q128JVS, U4 RP2040, U5 TXS0104ERGYR, Y1 ABLS-12.000MHZ-B4-T

Commit message: Updated strain gauge V2 to have a button
I need to update the button to be closer to ones we already have however.
Parts:
- removed J5: Conn_01x02, Connector_PinHeader_2.54mm:PinHeader_1x02_P2.54mm_Vertical, symbol Connector_Generic:Conn_01x02
- added SW2: SW_Push, Button_Switch_THT:SW_PUSH_6mm_H4.3mm, symbol Switch:SW_Push
Connections:
- net GND: now also SW2.1
- net ~{USB_BOOT}: now also SW2.2
Changed lines of the file:
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@@
+    (stroke (width 0) (type default))
+  )
+  (wire (pts (xy 27.94 91.44) (xy 43.18 91.44))
     (stroke (width 0) (type default))
   )
@@
     (stroke (width 0) (type default))
   )
-  (wire (pts (xy 44.45 95.25) (xy 44.45 96.52))
-    (stroke (width 0) (type default))
-  )
   (wire (pts (xy 186.69 62.23) (xy 186.69 49.53))
     (stroke (width 0) (type default))
@@
     (stroke (width 0) (type default))
   )
+  (wire (pts (xy 27.94 101.6) (xy 27.94 102.87))
+    (stroke (width 0) (type default))
+  )
   (wire (pts (xy 219.71 123.19) (xy 234.95 123.19))
     (stroke (width 0) (type default))
@@
     (stroke (width 0) (type default))
   )
+  (wire (pts (xy 43.18 91.44) (xy 43.18 92.71))
+    (stroke (width 0) (type default))
+  )
   (wire (pts (xy 102.87 97.79) (xy 119.38 97.79))
     (stroke (width 0) (type default))
@@
   )
   (wire (pts (xy 204.47 29.21) (xy 204.47 44.45))
-    (stroke (width 0) (type default))
-  )
-  (wire (pts (xy 43.18 95.25) (xy 44.45 95.25))
     (stroke (width 0) (type default))
   )
@@
     )
   )
-  (symbol (lib_id "Connector_Generic:Conn_01x02") (at 38.1 92.71 0) (mirror y) (unit 1)
-    (in_bom yes) (on_board yes) (dnp no)
-    (property "Reference" "J5" (at 36.83 88.9 0)
-      (effects (font (size 1.27 1.27)))
-    )
-    (property "Value" "Conn_01x02" (at 36.83 99.06 0)
-      (effects (font (size 1.27 1.27)))
-    )
-    (property "Footprint" "Connector_PinHeader_2.54mm:PinHeader_1x02_P2.54mm_Vertical" (at 38.1 92.71 0)
-      (effects (font (size 1.27 1.27)) hide)
-    )
-    (property "Datasheet" "~" (at 38.1 92.71 0)
-      (effects (font (size 1.27 1.27)) hide)
-    )
-    (property "Purchase Link" "https://www.digikey.com/en/products/detail/gct/BC020-02-A-0200-0300-L-G/12549946" (at 38.1 92.71 0)
-      (effects (font (size 1.27 1.27)) hide)
-    )
-    (pin "1")
-    (pin "2")
-    (instances
-      (project "Strain_Gauge"
-        (path "/25ee9722-784e-4ea5-b605-b90e2640812a"
-          (reference "J5") (unit 1)
-        )
-      )
-      (project "Strain_Gauge_V2"
-        (path "/9ba70739-c7bc-4186-9321-3785045f9d6e"
-          (reference "J7") (unit 1)
-        )
-        (path "/9ba70739-c7bc-4186-9321-3785045f9d6e/a7e84da9-b459-475d-86f6-7aea55b4eeae"
-          (reference "J7") (unit 1)
-        )
-      )
-    )
-  )
   (symbol (lib_id "Device:C") (at 224.79 34.29 0) (unit 1)
     (in_bom yes) (on_board yes) (dnp no)
@@
     )
   )
+  (symbol (lib_id "Switch:SW_Push") (at 27.94 96.52 90) (unit 1)
+    (in_bom yes) (on_board yes) (dnp no) (fields_autoplaced)
+    (property "Reference" "SW2" (at 29.21 95.885 90)
+      (effects (font (size 1.27 1.27)) (justify right))
+    )
+    (property "Value" "SW_Push" (at 29.21 98.425 90)
+      (effects (font (size 1.27 1.27)) (justify right))
+    )
+    (property "Footprint" "Button_Switch_THT:SW_PUSH_6mm_H4.3mm" (at 22.86 96.52 0)
+      (effects (font (size 1.27 1.27)) hide)
+    )
+    (property "Datasheet" "~" (at 22.86 96.52 0)
+      (effects (font (size 1.27 1.27)) hide)
+    )
+    (pin "1")
+    (pin "2")
+    (instances
+      (project "Strain_Gauge_V2"
+        (path "/9ba70739-c7bc-4186-9321-3785045f9d6e/a7e84da9-b459-475d-86f6-7aea55b4eeae"
+          (reference "SW2") (unit 1)
+        )
+      )
+    )
+  )
   (symbol (lib_id "power:+1V1") (at 167.64 27.94 0) (unit 1)
     (in_bom yes) (on_board yes) (dnp no)
@@
     )
   )
-  (symbol (lib_id "power:GND") (at 44.45 96.52 0) (unit 1)
-    (in_bom yes) (on_board yes) (dnp no)
-    (property "Reference" "#PWR01" (at 44.45 102.87 0)
-      (effects (font (size 1.27 1.27)) hide)
-    )
-    (property "Value" "GND" (at 44.577 100.9142 0)
-      (effects (font (size 1.27 1.27)))
-    )
-    (property "Footprint" "" (at 44.45 96.52 0)
-      (effects (font (size 1.27 1.27)) hide)
-    )
-    (property "Datasheet" "" (at 44.45 96.52 0)
-      (effects (font (size 1.27 1.27)) hide)
-    )
+  (symbol (lib_id "power:GND") (at 27.94 102.87 0) (unit 1)
+    (in_bom yes) (on_board yes) (dnp no)
+    (property "Reference" "#PWR01" (at 27.94 109.22 0)
+      (effects (font (size 1.27 1.27)) hide)
+    )
+    (property "Value" "GND" (at 28.067 107.2642 0)
+      (effects (font (size 1.27 1.27)))
+    )
+    (property "Footprint" "" (at 27.94 102.87 0)
+      (effects (font (size 1.27 1.27)) hide)
+    )
+    (property "Datasheet" "" (at 27.94 102.87 0)
+      (effects (font (size 1.27 1.27)) hide)
+    )

Commit message: Update footprint for part that we already have.
Technically footprint actually contains the name of the part here.
Parts:
- SW2: footprint Button_Switch_THT:SW_PUSH_6mm_H4.3mm -> Button_Switch_SMD:SW_SPST_B3U-1000P
Changed lines of the file:
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@@
       (effects (font (size 1.27 1.27)) (justify right))
     )
-    (property "Footprint" "Button_Switch_THT:SW_PUSH_6mm_H4.3mm" (at 22.86 96.52 0)
+    (property "Footprint" "Button_Switch_SMD:SW_SPST_B3U-1000P" (at 22.86 96.52 0)
       (effects (font (size 1.27 1.27)) hide)
     )
