File: Boards/Neo_Strain_Gauge/Strain_Gauge_V2/ADC.kicad_sch (KiCad schematic)
At the start: 11 parts, among them U6 ADS1274IPAPR, U7 MAX6102

Commit message: Update board to use two voltage references
This will be a "demo" for a two-reference board, next I will most likely
design one with a differential instrumentation amplifier before
having a new board with 4 instrumentation amplifiers and a single-ended
ADC involved.
Parts:
- added C35, C36: 10u, Capacitor_SMD:C_0402_1005Metric, symbol Device:C
- added U8: MAX6105, Package_TO_SOT_SMD:SOT-23, symbol Reference_Voltage:MAX6105
Connections:
- net GND: now also C35.2, C36.1, U8.3 (GND)
- new net +12V: C36.2, U8.1 (IN)
- new net +5VA: C35.1, U8.2 (OUT)
